File: pcb/filament dryer.kicad_pcb (KiCad board)
At the start: 2 copper layers, 65 x 65 mm, 24 parts, among them J1 Conn_01x02, J2 Screw_Terminal, J3 Conn_01x02, J4 Conn_01x02, J5 Conn_01x02, J6 Screw_Terminal, J7 Conn_01x02, J8 Conn_01x04, Q1 IRLZ44N, Q2 IRLZ44N, U1 SN65HVD230, U2 R-78E5.0-1.0

Commit message: PCB/CAD with README's
Parts:
- removed H2, H3: MountingHole, MountingHole:MountingHole_3.2mm_M3_Pad
- moved H1 54.0 mm to (26.0, 25.0)
- moved R3 31.2 mm to (52.1, 57.0), turned to 0 degrees
- moved R4 26.1 mm to (70.3, 46.5), turned to 180 degrees
- moved R7 15.5 mm to (27.5, 57.9)
- moved J2 13.4 mm to (69.3, 27.7), turned to 180 degrees
- moved R1 11.4 mm to (80.3, 57.0)
- moved J7 10.0 mm to (33.5, 52.2), turned to -90 degrees
- moved R6 8.98 mm to (34.8, 32.8), turned to -90 degrees
- moved U1 8.56 mm to (40.0, 53.5)
- moved J4 8.00 mm to (32.5, 24.4)
- moved J5 8.00 mm to (41.0, 24.4)
- moved J6 8.00 mm to (50.9, 27.0)
- moved J1 7.03 mm to (75.8, 24.4)
- moved J8 5.15 mm to (47.2, 52.5)
- moved J3 5.15 mm to (28.7, 38.4)
Routing:
- net +3V3: track 130.9 -> 89.5 mm
- net GND: track 16.9 -> 43.3 mm
- net fanEN: track 70.7 -> 57.5 mm
- net canTX: track 37.5 -> 26.6 mm
- net canRX: track 34.3 -> 24.8 mm
- net heaterEN: track 86.7 -> 94.6 mm
- net +5V: track 74.6 -> 67.0 mm
- net Net-(Q2-G): track 16.9 -> 12.3 mm
- net Net-(Q1-G): track 24.8 -> 28.9 mm
- net sda: track 20.4 -> 24.4 mm
- net canH: track 38.2 -> 42.2 mm
- net scl: track 12.0 -> 15.9 mm
- net Net-(J3-Pin_1): track 5.92 -> 9.63 mm
- net thermistor: track 6.44 -> 9.60 mm
- net Net-(J1-Pin_2): track 11.7 -> 9.84 mm
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Other:
- board text added: "- HE +"
- board text removed: "+ HE -"

Commit message: pcb update and firmware
Parts:
- moved R7 13.4 mm to (27.4, 44.5), turned to -90 degrees
- moved J7 3.21 mm to (32.9, 55.4), turned to 90 degrees
Connections:
- A1 pad 26: unconnected-(A1-GPIO20-Pad26) -> thermistor
Routing:
- net thermistor: track 9.60 -> 34.8 mm
- net GND: track 43.3 -> 27.0 mm
- net +3V3: track 89.5 -> 103.6 mm
