File: pcb/filament dryer.kicad_sch (KiCad schematic)
At the start: 19 parts, among them J1 Conn_01x02, J2 Screw_Terminal, J3 Conn_01x02_Pin, J4 Conn_01x02, J5 Conn_01x02, J6 Screw_Terminal, Q1 IRLZ44N, Q2 IRLZ44N, U1 SN65HVD230, U2 R-78E5.0-1.0

Commit message: pcb
Parts:
- removed J3: Conn_01x02_Pin, Connector_PinHeader_2.54mm:PinHeader_1x02_P2.54mm_Vertical, symbol Connector:Conn_01x02_Pin
- removed R5: 120Ω, Resistor_THT:R_Axial_DIN0309_L9.0mm_D3.2mm_P12.70mm_Horizontal, symbol Device:R
- added H1, H2, H3: MountingHole, MountingHole:MountingHole_3.2mm_M3_Pad, symbol Mechanical:MountingHole_Pad
- added J3, J7: Conn_01x02, Connector_JST:JST_XH_B2B-XH-A_1x02_P2.50mm_Vertical, symbol Connector_Generic:Conn_01x02
- added J8: Conn_01x04, Connector_PinSocket_2.54mm:PinSocket_1x04_P2.54mm_Vertical, symbol Connector_Generic:Conn_01x04
- added R7: 4.7KΩ, Resistor_THT:R_Axial_DIN0309_L9.0mm_D3.2mm_P12.70mm_Horizontal, symbol Device:R
- J1, J4, J5: LCSC Part (none) -> C378939
- Q1, Q2: footprint Package_TO_SOT_THT:TO-220-3_Vertical -> Package_TO_SOT_THT:TO-220-3_Horizontal_TabDown
Connections:
- net +3V3: now also J8.1 (Pin_1), R7.1
- net GND: now also H1.1, H2.1, H3.1, J7.2 (Pin_2), J8.3 (Pin_3); no longer A1.33 (AGND)
- net canH: now also J3.2 (Pin_2)
- net at R6.2: now also J3.1 (Pin_1)
- net sda: now reaches A1.4 (GPIO2)
- net sda: now also J8.2 (Pin_2)
- net scl: now reaches A1.5 (GPIO3)
- net scl: now also J8.4 (Pin_4)
- new net thermistor: J7.1 (Pin_1), R7.2
- no-connect marks 1 -> 25
Other:
- note added: "AHT21B sensor"
- note added: "mounting holes"
- note added: "thermistor"
- moved on the sheet: C1, C2, R3, R4, R6

Commit message: PCB/CAD with README's
Parts:
- removed H2, H3: MountingHole, MountingHole:MountingHole_3.2mm_M3_Pad, symbol Mechanical:MountingHole_Pad
Other:
- note added: "mounting hole"
- note removed: "mounting holes"
- moved on the sheet: H1

Commit message: pcb update and firmware
Connections:
- net thermistor: now also A1.26 (GPIO20)
- no-connect marks 25 -> 24
Changed lines of the file:
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@@
-	)
-	(no_connect
-		(at 166.37 59.69)
 	)
 	(no_connect
@@
 			(effects
 				(font
+					(size 1.27 1.27)
+				)
+				(justify left)
+				(hide yes)
+			)
+		)
+	)
+	(global_label "thermistor"
+		(shape input)
+		(at 166.37 59.69 0)
+		(fields_autoplaced yes)
+		(effects
+			(font
+				(size 1.27 1.27)
+			)
+			(justify left)
+		)
+		(property "Intersheetrefs" "${INTERSHEET_REFS}"
+			(at 179.0918 59.69 0)
+			(effects
+				(font
